Commit message: marker thickness option

File: table/urdf/table.urdf.xacro (robot description, xacro)
@@ -17,4 +17,5 @@
     <xacro:arg name="marker_id" default="0"/>
     <xacro:arg name="marker_pos" default="2"/>
+    <xacro:arg name="marker_thickness" default="0.001"/>
     <xacro:property name="surface_size_x" value="$(arg surface_size_x)"/>
     <xacro:property name="surface_size_y" value="$(arg surface_size_y)"/>
@@ -33,4 +34,5 @@
     <xacro:property name="marker_id" value="$(arg marker_id)"/>
     <xacro:property name="marker_pos" value="$(arg marker_pos)"/>
+    <xacro:property name="marker_thickness" value="$(arg marker_thickness)"/>
     <material name="${surface_gazebo_color}">
         <color rgba="1.0 1.0 1.0 1.0"/>
@@ -146,5 +148,5 @@
     <joint name="aruco_front_joint" type="fixed">
       <parent link="${surface_name}"/>
-      <origin xyz="0 0 ${surface_size_z/2 + 0.001}" rpy="0 0 0"/>
+      <origin xyz="0 0 ${surface_size_z/2 + 1e-5 + marker_thickness}" rpy="0 0 0"/>
       <child link="fiducial_${marker_id}"/>
     </joint>
@@ -193,5 +195,5 @@
     <joint name="aruco_nw_joint" type="fixed">
       <parent link="${surface_name}"/>
-      <origin xyz="${-surface_size_x/2} ${surface_size_y/2 - marker_size/2} ${surface_size_z/2 - marker_size/2}" rpy="0 1.5708 0"/>
+      <origin xyz="${-(surface_size_x/2 + 1e-5 + marker_thickness)} ${surface_size_y/2 - marker_size/2} ${surface_size_z/2 - marker_size/2}" rpy="0 1.5708 0"/>
       <child link="fiducial_${marker_id}"/>
     </joint>
@@ -240,5 +242,5 @@
     <joint name="aruco_n_joint" type="fixed">
       <parent link="${surface_name}"/>
-      <origin xyz="${-surface_size_x/2} 0 ${surface_size_z/2 - marker_size/2}" rpy="0 1.5708 0"/>
+      <origin xyz="${-surface_size_x/2 + 1e-5 + marker_thickness} 0 ${surface_size_z/2 - marker_size/2}" rpy="0 1.5708 0"/>
       <child link="fiducial_${marker_id}"/>
     </joint>

Commit message: add useful links

File: table/urdf/table.urdf.xacro (robot description, xacro)
@@ -68,4 +68,16 @@
         <material>${surface_gazebo_color}</material>
     </gazebo>
+    <link name="table_base_footprint"></link>
+    <joint name="table_base_footprint_joint" type="fixed">
+        <parent link="${surface_name}"/>
+        <origin rpy="0.0 0.0 0.0" xyz="0 0 ${-surface_high}"/>
+        <child link="table_base_footprint"/>
+    </joint>
+    <link name="${surface_name}_top"></link>
+    <joint name="${surface_name}_top_joint" type="fixed">
+        <parent link="${surface_name}"/>
+        <origin rpy="0.0 0.0 0.0" xyz="0 0 ${surface_size_z/2}"/>
+        <child link="${surface_name}_top"/>
+    </joint>
     <!-- LEGS -->
     <xacro:macro name="table_leg" params="name">

Commit message: tables corrected as per definition of surface_high

File: table/urdf/table.urdf.xacro (robot description, xacro)
@@ -17,5 +17,5 @@
     <xacro:arg name="marker_id" default="0"/>
     <xacro:arg name="marker_pos" default="2"/>
-    <xacro:arg name="marker_thickness" default="0.001"/>
+    <xacro:arg name="marker_thickness" default="0.00001"/>
     <xacro:property name="surface_size_x" value="$(arg surface_size_x)"/>
     <xacro:property name="surface_size_y" value="$(arg surface_size_y)"/>
@@ -41,5 +41,5 @@
         <color rgba=".3 .3 .3 1.0"/>
     </material>
-    <origin rpy="0 0 0" xyz="0 0 ${surface_high}"/>
+    <origin rpy="0 0 0" xyz="0 0 ${surface_high-surface_size_z/2}"/>
     <link name="${surface_name}">
         <inertial>
@@ -71,5 +71,5 @@
     <joint name="table_base_footprint_joint" type="fixed">
         <parent link="${surface_name}"/>
-        <origin rpy="0.0 0.0 0.0" xyz="0 0 ${-surface_high}"/>
+        <origin rpy="0.0 0.0 0.0" xyz="0 0 ${-surface_high+(surface_size_z/2)}"/>
         <child link="table_base_footprint"/>
     </joint>
@@ -85,11 +85,11 @@
         <inertial>
             <mass value="${leg_mass}" />
-            <inertia    ixx="${0.083 * leg_mass * (3*0.02*0.02 + surface_high*surface_high)}"  ixy="0.0"  ixz="0.0"
-                        iyy="${0.083 * leg_mass * (3*0.02*0.02 + surface_high*surface_high)}"  iyz="0.0"
+            <inertia    ixx="${0.083 * leg_mass * (3*0.02*0.02 + (surface_high - surface_size_z)*(surface_high - surface_size_z))}"  ixy="0.0"  ixz="0.0"
+                        iyy="${0.083 * leg_mass * (3*0.02*0.02 + (surface_high - surface_size_z)*(surface_high - surface_size_z))}"  iyz="0.0"
                         izz="${0.5 * leg_mass * 0.02 * 0.02}" />
         </inertial>
         <collision>
             <geometry>
-                <cylinder radius="0.02" length="${surface_high}"/>
+                <cylinder radius="0.02" length="${surface_high - surface_size_z}"/>
             </geometry>
         </collision>
@@ -97,5 +97,5 @@
             <origin xyz="0 0 0" rpy="0 0 0" />
             <geometry>
-                <cylinder radius="0.02" length="${surface_high}"/>
+                <cylinder radius="0.02" length="${surface_high - surface_size_z}"/>
             </geometry>
             <material name="${leg_gazebo_color}"/>
@@ -141,7 +141,7 @@
     <link name="fiducial_${marker_id}">
       <visual>
-        <origin xyz="0 0 0" rpy="0 0 0" />
-        <geometry>
-          <box size="${marker_size} ${marker_size} 1e-5"/>
+        <origin xyz="0 0 ${-marker_thickness/2}" rpy="0 0 0" />
+        <geometry>
+          <box size="${marker_size} ${marker_size} ${marker_thickness}"/>
         </geometry>
         <material name="aruco_color_rviz">
@@ -150,9 +150,9 @@
       </visual>
       <collision>
-        <origin xyz="0 0 0" rpy="0 0 0" />
+        <origin xyz="0 0 ${-marker_thickness/2}" rpy="0 0 0" />
         <laser_retro>0</laser_retro>
         <max_contacts>10</max_contacts>
         <geometry>
-          <box size="${marker_size} ${marker_size} 1e-5"/>
+          <box size="${marker_size} ${marker_size} ${marker_thickness}"/>
         </geometry>
       </collision>
@@ -160,5 +160,5 @@
     <joint name="aruco_front_joint" type="fixed">
       <parent link="${surface_name}"/>
-      <origin xyz="0 0 ${surface_size_z/2 + 1e-5 + marker_thickness}" rpy="0 0 0"/>
+      <origin xyz="0 0 ${surface_size_z/2 + marker_thickness}" rpy="0 0 0"/>
       <child link="fiducial_${marker_id}"/>
     </joint>
@@ -190,5 +190,5 @@
         <origin xyz="0 0 0" rpy="0 0 0" />
         <geometry>
-          <box size="${marker_size} ${marker_size} 1e-5"/>
+          <box size="${marker_size} ${marker_size} ${marker_thickness}"/>
         </geometry>
         <material name="aruco_color_rviz">
@@ -201,5 +201,5 @@
         <max_contacts>10</max_contacts>
         <geometry>
-          <box size="${marker_size} ${marker_size} 1e-5"/>
+          <box size="${marker_size} ${marker_size} ${marker_thickness}"/>
         </geometry>
       </collision>
@@ -207,5 +207,5 @@
     <joint name="aruco_nw_joint" type="fixed">
       <parent link="${surface_name}"/>
-      <origin xyz="${-(surface_size_x/2 + 1e-5 + marker_thickness)} ${surface_size_y/2 - marker_size/2} ${surface_size_z/2 - marker_size/2}" rpy="0 1.5708 0"/>
+      <origin xyz="${-(surface_size_x/2 + marker_thickness/2)} ${surface_size_y/2 - marker_size/2} ${surface_size_z/2 - marker_size/2}" rpy="0 1.5708 0"/>
       <child link="fiducial_${marker_id}"/>
     </joint>
@@ -237,5 +237,5 @@
         <origin xyz="0 0 0" rpy="0 0 0" />
         <geometry>
-          <box size="${marker_size} ${marker_size} 1e-5"/>
+          <box size="${marker_size} ${marker_size} ${marker_thickness}"/>
         </geometry>
         <material name="aruco_color_rviz">
@@ -248,5 +248,5 @@
         <max_contacts>10</max_contacts>
         <geometry>
-          <box size="${marker_size} ${marker_size} 1e-5"/>
+          <box size="${marker_size} ${marker_size} ${marker_thickness}"/>
         </geometry>
       </collision>
@@ -254,5 +254,5 @@
     <joint name="aruco_n_joint" type="fixed">
       <parent link="${surface_name}"/>
-      <origin xyz="${-surface_size_x/2 + 1e-5 + marker_thickness} 0 ${surface_size_z/2 - marker_size/2}" rpy="0 1.5708 0"/>
+      <origin xyz="${-surface_size_x/2 + marker_thickness} 0 ${surface_size_z/2 - marker_size/2}" rpy="0 1.5708 0"/>
       <child link="fiducial_${marker_id}"/>
     </joint>

File: table/urdf/table_inverted.urdf.xacro (robot description, xacro)
@@ -16,5 +16,5 @@
     <xacro:arg name="marker_id" default="0"/>
     <xacro:arg name="marker_pos" default="2"/>
-    <xacro:arg name="marker_thickness" default="0.001"/>
+    <xacro:arg name="marker_thickness" default="0.00001"/>
     <xacro:property name="surface_size_x" value="$(arg surface_size_x)"/>
     <xacro:property name="surface_size_y" value="$(arg surface_size_y)"/>
@@ -40,5 +40,5 @@
         <color rgba=".3 .3 .3 1.0"/>
     </material>
-    <origin rpy="0 0 0" xyz="0 0 ${surface_high + surface_size_z/2 + 1e-5 + marker_thickness}"/>
+    <origin rpy="0 0 0" xyz="0 0 ${surface_high + marker_thickness}"/>
     <link name="${surface_name}">
         <inertial>
@@ -70,5 +70,5 @@
     <joint name="table_base_footprint_joint" type="fixed">
         <parent link="${surface_name}"/>
-        <origin rpy="0.0 0.0 0.0" xyz="0 0 ${-surface_high}"/>
+        <origin rpy="0.0 0.0 0.0" xyz="0 0 ${-surface_high+(surface_size_z/2)}"/>
         <child link="table_base_footprint"/>
     </joint>
@@ -84,11 +84,11 @@
         <inertial>
             <mass value="${leg_mass}" />
-            <inertia    ixx="${0.083 * leg_mass * (3*0.02*0.02 + surface_high*surface_high)}"  ixy="0.0"  ixz="0.0"
-                        iyy="${0.083 * leg_mass * (3*0.02*0.02 + surface_high*surface_high)}"  iyz="0.0"
+            <inertia    ixx="${0.083 * leg_mass * (3*0.02*0.02 + (surface_high - surface_size_z)*(surface_high - surface_size_z))}"  ixy="0.0"  ixz="0.0"
+                        iyy="${0.083 * leg_mass * (3*0.02*0.02 + (surface_high - surface_size_z)*(surface_high - surface_size_z))}"  iyz="0.0"
                         izz="${0.5 * leg_mass * 0.02 * 0.02}" />
         </inertial>
         <collision>
             <geometry>
-                <cylinder radius="0.02" length="${surface_high}"/>
+                <cylinder radius="0.02" length="${surface_high - surface_size_z}"/>
             </geometry>
         </collision>
@@ -96,5 +96,5 @@
             <origin xyz="0 0 0" rpy="0 0 0" />
             <geometry>
-                <cylinder radius="0.02" length="${surface_high}"/>
+                <cylinder radius="0.02" length="${surface_high - surface_size_z}"/>
             </geometry>
             <material name="${leg_gazebo_color}"/>
@@ -139,7 +139,7 @@
     <link name="fiducial_${marker_id}">
       <visual>
-        <origin xyz="0 0 0" rpy="0 0 0" />
+        <origin xyz="0 0 ${-marker_thickness/2}" rpy="0 0 0" />
         <geometry>
-          <box size="${marker_size} ${marker_size} 1e-5"/>
+          <box size="${marker_size} ${marker_size} ${marker_thickness}"/>
         </geometry>
         <material name="aruco_color_rviz">
@@ -148,9 +148,9 @@
       </visual>
       <collision>
-        <origin xyz="0 0 0" rpy="0 0 0" />
+        <origin xyz="0 0 ${-marker_thickness/2}" rpy="0 0 0" />
         <laser_retro>0</laser_retro>
         <max_contacts>10</max_contacts>
         <geometry>
-          <box size="${marker_size} ${marker_size} 1e-5"/>
+          <box size="${marker_size} ${marker_size} ${marker_thickness}"/>
         </geometry>
       </collision>
@@ -158,5 +158,5 @@
     <joint name="aruco_front_joint" type="fixed">
       <child link="${surface_name}"/>
-      <origin xyz="0 0 -${surface_size_z/2 + 1e-5 + marker_thickness}" rpy="0 0 0"/>
+      <origin xyz="0 0 ${-surface_size_z/2 - marker_thickness}" rpy="0 0 0"/>
       <parent link="fiducial_${marker_id}"/>
     </joint>

Commit message: simplekeyboard and table updated to accomodate it

File: table/urdf/table.urdf.xacro (robot description, xacro)
@@ -18,4 +18,10 @@
     <xacro:arg name="marker_pos" default="2"/>
     <xacro:arg name="marker_thickness" default="0.00001"/>
+<!--   keyboard on top the table   -->
+    <xacro:arg name="keyboard" default="false"/>
+    <xacro:arg name="keyboard_parent" default="surface_top"/>
+    <xacro:arg name="keyboard_x" default="0"/>
+    <xacro:arg name="keyboard_y" default="0"/>
+    <xacro:arg name="keyboard_z" default="0"/>
     <xacro:property name="surface_size_x" value="$(arg surface_size_x)"/>
     <xacro:property name="surface_size_y" value="$(arg surface_size_y)"/>
@@ -35,4 +41,10 @@
     <xacro:property name="marker_pos" value="$(arg marker_pos)"/>
     <xacro:property name="marker_thickness" value="$(arg marker_thickness)"/>
+    <!-- keyboard related -->
+    <xacro:property name="keyboard" value="$(arg keyboard)"/>
+    <xacro:property name="keyboard_parent" value="$(arg keyboard_parent)"/>
+    <xacro:property name="keyboard_x" value="$(arg keyboard_x)"/>
+    <xacro:property name="keyboard_y" value="$(arg keyboard_y)"/>
+    <xacro:property name="keyboard_z" value="$(arg keyboard_z)"/>
     <material name="${surface_gazebo_color}">
         <color rgba="1.0 1.0 1.0 1.0"/>
@@ -135,4 +147,11 @@
         <child link="back_left_leg"/>
     </joint>
+        <!--   KEYBOARD   -->
+    <xacro:if value="${keyboard}">
+        <xacro:include filename="$(find iit_gazebo_worlds_pkg)/simpleKeyboard/urdf/keyboard_macro.urdf.xacro" />
+        <xacro:simple_keyboard parent="surface_top">
+            <origin xyz="${keyboard_x} ${keyboard_y} ${keyboard_z}" rpy="0 0 0" />
+        </xacro:simple_keyboard>
+    </xacro:if>
     <!--  ********************************* Links for arucos **********************************************************  -->
     <xacro:if value="${markers}">
