Commit message: virtual keyboard in development

File: simpleKeyboard/urdf/keyboard.urdf.xacro (robot description, xacro)
@@ -2,5 +2,4 @@
 <robot xmlns:xacro="http://ros.org/wiki/xacro" name="keyboard">
     <xacro:include filename="$(find iit_gazebo_worlds_pkg)/simpleKeyboard/urdf/keyboard_macro.urdf.xacro" />
-    <xacro:include filename="$(find iit_gazebo_worlds_pkg)/simpleKeyboard/urdf/properties.urdf.xacro" />
     <link name="world"></link>
     <xacro:simple_keyboard parent="world">

File: simpleKeyboard/urdf/properties.urdf.xacro (robot description, xacro)
@@ -10,5 +10,6 @@
     <xacro:property name="kd" value="1"/>
     <xacro:property name="key_names"        value="${['z_neg',    'x_pos',      'z_pos',      'y_pos',       'x_neg',    'y_neg']}" />
-    <xacro:property name="key_colors"       value="${['dark_blue', 'light_red', 'light_blue', 'light_green', 'dark_red', 'dark_green']}" />
+<!--    <xacro:property name="key_colors"       value="${['dark_blue', 'light_red', 'light_blue', 'light_green', 'dark_red', 'dark_green']}" />-->
+    <xacro:property name="key_colors"       value="${['white', 'white', 'white', 'white', 'white', 'white']}" />
     <xacro:property name="key_colors_gazebo"       value="${['Gazebo/Blue', 'Gazebo/Red', 'Gazebo/Blue', 'Gazebo/Green', 'Gazebo/Red', 'Gazebo/Green']}" />
     <xacro:property name="top_right_corner_x" value="${keyboard_rows/2 * key_size_x}"/>
@@ -32,3 +33,9 @@
         <color rgba="0.0 0.0 0.5 1"/>
     </material>
+    <material name="trasparent">
+        <color rgba="0.0 0.0 0.0 0"/>
+    </material>
+    <material name="white">
+        <color rgba="1.0 1.0 1.0 1"/>
+    </material>
 </robot>
