Commit message: virtual keyboard on the table!

File: simpleKeyboard/urdf/properties.urdf.xacro (robot description, xacro)
@@ -1,16 +1,22 @@
 <!--<?xml version="1.0"?>-->
 <robot  xmlns:xacro="http://ros.org/wiki/xacro">
-    <xacro:property name="keyboard_name" value="keyboard"/>
-    <xacro:property name="key_size_x" value="0.1"/>
-    <xacro:property name="key_size_y" value="0.1"/>
-    <xacro:property name="key_size_z" value="0.001"/>
-    <xacro:property name="keyboard_rows" value="2"/>
-    <xacro:property name="keyboard_cols" value="3"/>
+    <xacro:arg name="keyboard_name" default="keyboard"/>
+    <xacro:arg name="key_size_x" default="0.1"/>
+    <xacro:arg name="key_size_y" default="0.1"/>
+    <xacro:arg name="key_size_z" default="0.001"/>
+    <xacro:arg name="keyboard_rows" default="4"/>
+    <xacro:arg name="keyboard_cols" default="3"/>
+    <xacro:property name="keyboard_name" value="$(arg keyboard_name)"/>
+    <xacro:property name="key_size_x" value="$(arg key_size_x)"/>
+    <xacro:property name="key_size_y" value="$(arg key_size_y)"/>
+    <xacro:property name="key_size_z" value="$(arg key_size_z)"/>
+    <xacro:property name="keyboard_rows" value="$(arg keyboard_rows)"/>
+    <xacro:property name="keyboard_cols" value="$(arg keyboard_cols)"/>
     <xacro:property name="kp" value="1e13"/>
     <xacro:property name="kd" value="1"/>
-    <xacro:property name="key_names"        value="${['z_neg',    'x_pos',      'z_pos',      'y_pos',       'x_neg',    'y_neg']}" />
+    <xacro:property name="key_names"        value="${['z_neg',    'x_pos',      'z_pos',      'y_pos',       'x_neg',    'y_neg', 'yaw_pos', 'yaw_neg', 'stop' ,'open_gripper', 'close_gripper', 'none']}" />
 <!--    <xacro:property name="key_colors"       value="${['dark_blue', 'light_red', 'light_blue', 'light_green', 'dark_red', 'dark_green']}" />-->
-    <xacro:property name="key_colors"       value="${['white', 'white', 'white', 'white', 'white', 'white']}" />
-    <xacro:property name="key_colors_gazebo"       value="${['Gazebo/Blue', 'Gazebo/Red', 'Gazebo/Blue', 'Gazebo/Green', 'Gazebo/Red', 'Gazebo/Green']}" />
+    <xacro:property name="key_colors"       value="${['white', 'white', 'white', 'white', 'white', 'white', 'white', 'white', 'white', 'white', 'white', 'white']}" />
+    <xacro:property name="key_colors_gazebo"       value="${['Gazebo/Blue', 'Gazebo/Red', 'Gazebo/Blue', 'Gazebo/Green', 'Gazebo/Red', 'Gazebo/Green', 'Gazebo/Blue', 'Gazebo/Blue', 'Gazebo/FlatBlack', 'Gazebo/DarkGrey', 'Gazebo/DarkGrey', 'Gazebo/FlatBlack']}" />
     <xacro:property name="top_right_corner_x" value="${keyboard_rows/2 * key_size_x}"/>
     <xacro:property name="top_right_corner_y" value="${keyboard_cols/2 * key_size_y}"/>

File: table/urdf/table.urdf.xacro (robot description, xacro)
@@ -20,4 +20,9 @@
 <!--   keyboard on top the table   -->
     <xacro:arg name="keyboard" default="false"/>
+    <xacro:arg name="key_size_x" default="0.1"/>
+    <xacro:arg name="key_size_y" default="0.1"/>
+    <xacro:arg name="key_size_z" default="0.0001"/>
+    <xacro:arg name="keyboard_rows" default="3"/>
+    <xacro:arg name="keyboard_cols" default="3"/>
     <xacro:arg name="keyboard_parent" default="surface_top"/>
     <xacro:arg name="keyboard_x" default="0"/>
@@ -43,4 +48,9 @@
     <!-- keyboard related -->
     <xacro:property name="keyboard" value="$(arg keyboard)"/>
+    <xacro:property name="key_size_x" value="$(arg key_size_x)"/>
+    <xacro:property name="key_size_y" value="$(arg key_size_y)"/>
+    <xacro:property name="key_size_z" value="$(arg key_size_z)"/>
+    <xacro:property name="keyboard_rows" value="$(arg keyboard_rows)"/>
+    <xacro:property name="keyboard_cols" value="$(arg keyboard_cols)"/>
     <xacro:property name="keyboard_parent" value="$(arg keyboard_parent)"/>
     <xacro:property name="keyboard_x" value="$(arg keyboard_x)"/>

Commit message: keyboard as in humanoids23 exp

File: simpleKeyboard/urdf/properties.urdf.xacro (robot description, xacro)
@@ -15,5 +15,5 @@
     <xacro:property name="kp" value="1e13"/>
     <xacro:property name="kd" value="1"/>
-    <xacro:property name="key_names"        value="${['z_neg',    'x_pos',      'z_pos',      'y_pos',       'x_neg',    'y_neg', 'yaw_pos', 'yaw_neg', 'stop' ,'open_gripper', 'close_gripper', 'none']}" />
+    <xacro:property name="key_names"        value="${['none_0', 'yaw_pos', 'yaw_neg', 'z_neg', 'x_pos',  'z_pos',  'y_pos',  'x_neg', 'y_neg', 'none_9','open_gripper', 'close_gripper']}" />
 <!--    <xacro:property name="key_colors"       value="${['dark_blue', 'light_red', 'light_blue', 'light_green', 'dark_red', 'dark_green']}" />-->
     <xacro:property name="key_colors"       value="${['white', 'white', 'white', 'white', 'white', 'white', 'white', 'white', 'white', 'white', 'white', 'white']}" />

Commit message: conf for exp

File: simpleKeyboard/urdf/properties.urdf.xacro (robot description, xacro)
@@ -15,5 +15,6 @@
     <xacro:property name="kp" value="1e13"/>
     <xacro:property name="kd" value="1"/>
-    <xacro:property name="key_names"        value="${['none_0', 'yaw_pos', 'yaw_neg', 'z_neg', 'x_pos',  'z_pos',  'y_pos',  'x_neg', 'y_neg', 'none_9','open_gripper', 'close_gripper']}" />
+<!--    <xacro:property name="key_names"        value="${['none_0', 'yaw_pos', 'yaw_neg', 'z_neg', 'x_pos',  'z_pos',  'y_pos',  'x_neg', 'y_neg', 'none_9','open_gripper', 'close_gripper']}" />-->
+    <xacro:property name="key_names"        value="${['z_neg', 'x_pos',  'z_pos',  'y_pos',  'x_neg', 'y_neg']}" />
 <!--    <xacro:property name="key_colors"       value="${['dark_blue', 'light_red', 'light_blue', 'light_green', 'dark_red', 'dark_green']}" />-->
     <xacro:property name="key_colors"       value="${['white', 'white', 'white', 'white', 'white', 'white', 'white', 'white', 'white', 'white', 'white', 'white']}" />

Commit message: new update conf

File: simpleKeyboard/urdf/properties.urdf.xacro (robot description, xacro)
@@ -15,6 +15,6 @@
     <xacro:property name="kp" value="1e13"/>
     <xacro:property name="kd" value="1"/>
-<!--    <xacro:property name="key_names"        value="${['none_0', 'yaw_pos', 'yaw_neg', 'z_neg', 'x_pos',  'z_pos',  'y_pos',  'x_neg', 'y_neg', 'none_9','open_gripper', 'close_gripper']}" />-->
-    <xacro:property name="key_names"        value="${['z_neg', 'x_pos',  'z_pos',  'y_pos',  'x_neg', 'y_neg']}" />
+    <xacro:property name="key_names"        value="${['none_0', 'yaw_pos', 'yaw_neg', 'z_neg', 'x_pos',  'z_pos',  'y_pos',  'x_neg', 'y_neg', 'none_9','open_gripper', 'close_gripper']}" />
+<!--    <xacro:property name="key_names"        value="${['z_neg', 'x_pos',  'z_pos',  'y_pos',  'x_neg', 'y_neg']}" /> -->
 <!--    <xacro:property name="key_colors"       value="${['dark_blue', 'light_red', 'light_blue', 'light_green', 'dark_red', 'dark_green']}" />-->
     <xacro:property name="key_colors"       value="${['white', 'white', 'white', 'white', 'white', 'white', 'white', 'white', 'white', 'white', 'white', 'white']}" />

Commit message: donuts

File: simpleKeyboard/urdf/properties.urdf.xacro (robot description, xacro)
@@ -16,5 +16,5 @@
     <xacro:property name="kd" value="1"/>
     <xacro:property name="key_names"        value="${['none_0', 'yaw_pos', 'yaw_neg', 'z_neg', 'x_pos',  'z_pos',  'y_pos',  'x_neg', 'y_neg', 'none_9','open_gripper', 'close_gripper']}" />
-<!--    <xacro:property name="key_names"        value="${['z_neg', 'x_pos',  'z_pos',  'y_pos',  'x_neg', 'y_neg']}" /> -->
+<!-- <xacro:property name="key_names"        value="${['z_neg', 'x_pos',  'z_pos',  'y_pos',  'x_neg', 'y_neg']}" /> -->
 <!--    <xacro:property name="key_colors"       value="${['dark_blue', 'light_red', 'light_blue', 'light_green', 'dark_red', 'dark_green']}" />-->
     <xacro:property name="key_colors"       value="${['white', 'white', 'white', 'white', 'white', 'white', 'white', 'white', 'white', 'white', 'white', 'white']}" />

Commit message: comments

File: simpleKeyboard/urdf/properties.urdf.xacro (robot description, xacro)
@@ -15,6 +15,6 @@
     <xacro:property name="kp" value="1e13"/>
     <xacro:property name="kd" value="1"/>
-<!--    <xacro:property name="key_names"        value="${['none_0', 'yaw_pos', 'yaw_neg', 'z_neg', 'x_pos',  'z_pos',  'y_pos',  'x_neg', 'y_neg', 'none_9','open_gripper', 'close_gripper']}" />-->
-    <xacro:property name="key_names"        value="${['z_neg', 'x_pos',  'z_pos',  'y_pos',  'x_neg', 'y_neg']}" />
+    <xacro:property name="key_names"        value="${['none_0', 'yaw_pos', 'yaw_neg', 'z_neg', 'x_pos',  'z_pos',  'y_pos',  'x_neg', 'y_neg', 'none_9','open_gripper', 'close_gripper']}" />
+<!-- <xacro:property name="key_names"        value="${['z_neg', 'x_pos',  'z_pos',  'y_pos',  'x_neg', 'y_neg']}" /> -->
 <!--    <xacro:property name="key_colors"       value="${['dark_blue', 'light_red', 'light_blue', 'light_green', 'dark_red', 'dark_green']}" />-->
     <xacro:property name="key_colors"       value="${['white', 'white', 'white', 'white', 'white', 'white', 'white', 'white', 'white', 'white', 'white', 'white']}" />
