Commit message: static option, publish descr and tf if static

File: genericShapes/urdf/cylinder.urdf.xacro (robot description, xacro)
@@ -5,4 +5,5 @@
     <xacro:arg name="radius" default="0.5361"/>
     <xacro:arg name="mass" default="2"/>
+    <xacro:arg name="static" default="false"/>
     <xacro:arg name="r" default="0"/>
     <xacro:arg name="g" default="0"/>
@@ -18,4 +19,5 @@
     <xacro:property name="radius" value="$(arg radius)"/>
     <xacro:property name="mass" value="$(arg mass)"/>
+    <xacro:property name="static" value="$(arg static)"/>
     <xacro:property name="r" value="$(arg r)"/>
     <xacro:property name="g" value="$(arg g)"/>
@@ -57,4 +59,7 @@
 		</collision>
 	</link>
+    <gazebo>
+        <static>${static}</static>
+    </gazebo>
     <gazebo reference="${name}_link">
         <mu1>${mu1}</mu1>

Commit message: no _link easier to handle tf

File: genericShapes/urdf/cylinder.urdf.xacro (robot description, xacro)
@@ -29,5 +29,5 @@
     <xacro:property name="mu1" value="$(arg mu1)"/>
     <xacro:property name="mu2" value="$(arg mu2)"/>
-    <link name="${name}_link">
+    <link name="${name}">
 		<inertial>
             <mass value="${mass}" />
@@ -62,5 +62,5 @@
         <static>${static}</static>
     </gazebo>
-    <gazebo reference="${name}_link">
+    <gazebo reference="${name}">
         <mu1>${mu1}</mu1>
         <mu2>${mu2}</mu2>

File: genericShapes/urdf/sphere.urdf.xacro (robot description, xacro)
@@ -27,5 +27,5 @@
     <xacro:property name="mu1" value="$(arg mu1)"/>
     <xacro:property name="mu2" value="$(arg mu2)"/>
-    <link name="${name}_link">
+    <link name="${name}">
         <inertial>
             <mass value="${mass}" />
@@ -59,5 +59,5 @@
         <static>${static}</static>
     </gazebo>
-    <gazebo reference="${name}_link">
+    <gazebo reference="${name}">
         <mu1>${mu1}</mu1>
         <mu2>${mu2}</mu2>
